File: scheme/light_mul.kicad_pcb (KiCad board)
At the start: 2 copper layers, 100 parts, among them J1 Screw_Terminal_01x04 (buttons), J2 Conn_01x06_Male (programmer), J3 Screw_Terminal_01x06 (output), J4 Conn_01x02_Male (i2c), J5 Conn_01x02_Male (Jumper), J6 Conn_01x03_Male (Indicators), J7 Screw_Terminal_01x02 (power), Q1 IRF8308M, Q2 IRF8308M, Q3 IRF8308M, SW1 SW_Push (reset), U1 L7805, U2 ATmega8A-PU

Commit message: scheme: change routes widths
And avoid between pins routes
Parts:
- removed the C1 at (247.2, 122.8)
- removed the C1 at (247.2, 17.8)
- removed the C1 at (97.2, 122.8)
- removed the C2 at (247.2, 131.7)
- removed the C2 at (247.2, 26.7)
- removed the C2 at (97.2, 131.7)
- removed the J1 at (249.7, 162.2)
- removed the J1 at (249.7, 57.1)
- removed the J1 at (99.7, 162.2)
- removed the J2 at (207.8, 199.0)
- removed the J2 at (207.8, 94.0)
- removed the J2 at (57.8, 199.0)
- removed the J3 at (160.8, 181.2)
- removed the J3 at (160.8, 76.2)
- removed the J3 at (10.8, 181.2)
- removed the J4 at (223.0, 145.6)
- removed the J4 at (223.0, 40.6)
- removed the J4 at (73.0, 145.6)
- removed the J5 at (201.4, 199.0)
- removed the J5 at (201.4, 94.0)
- removed the J5 at (51.4, 199.0)
- removed the J6 at (196.4, 141.8)
- removed the J6 at (196.4, 36.8)
- removed the J6 at (46.4, 141.8)
- removed the J7 at (219.2, 124.0)
- removed the J7 at (219.2, 19.1)
- removed the J7 at (69.2, 124.0)
- removed the Q1 at (173.5, 183.7)
- removed the Q1 at (173.5, 78.7)
- removed the Q1 at (23.5, 183.7)
- removed the Q2 at (173.5, 169.8)
- removed the Q2 at (173.5, 64.8)
- removed the Q2 at (23.5, 169.8)
- removed the Q3 at (173.5, 155.8)
- removed the Q3 at (173.5, 50.8)
- removed the Q3 at (23.5, 155.8)
- removed the R1 at (223.0, 183.1)
- removed the R1 at (223.0, 78.1)
- removed the R1 at (73.0, 183.1)
- removed the R10 at (181.1, 157.1)
- removed the R10 at (181.1, 52.1)
- removed the R10 at (31.1, 157.1)
- removed the R2 at (228.1, 159.0)
- removed the R2 at (228.1, 54.0)
- removed the R2 at (78.1, 159.0)
- removed the R3 at (228.1, 153.3)
- removed the R3 at (228.1, 48.3)
- removed the R3 at (78.1, 153.3)
- removed the R4 at (228.1, 148.2)
- removed the R4 at (228.1, 43.2)
- removed the R4 at (78.1, 148.2)
- removed the R5 at (181.1, 185.0)
- removed the R5 at (181.1, 80.0)
- removed the R5 at (31.1, 185.0)
- removed the R6 at (184.9, 192.6)
- removed the R6 at (184.9, 87.6)
- removed the R6 at (34.9, 192.6)
- removed the R7 at (195.1, 168.5)
- removed the R7 at (195.1, 63.5)
- removed the R7 at (45.1, 168.5)
- removed the R8 at (181.1, 171.0)
- removed the R8 at (181.1, 66.0)
- removed the R8 at (31.1, 171.0)
- removed the R9 at (195.1, 157.1)
- removed the R9 at (195.1, 52.1)
- removed the R9 at (45.1, 157.1)
- removed the SW1 at (196.4, 182.5)
- removed the SW1 at (196.4, 77.5)
- removed the SW1 at (46.4, 182.5)
- removed the U1 at (234.5, 124.0)
- removed the U1 at (234.5, 19.1)
- removed the U1 at (84.5, 124.0)
- removed the U2 at (207.6, 143.4)
- removed the U2 at (207.6, 38.4)
- removed the U2 at (57.6, 143.4)
- added C1: 3.3uF, Capacitor_THT:C_Disc_D5.1mm_W3.2mm_P5.00mm, F.Cu at (122.2, 127.8)
- added C1: 3.3uF, Capacitor_THT:C_Disc_D5.1mm_W3.2mm_P5.00mm, F.Cu at (262.2, 127.8)
- added C1: 3.3uF, Capacitor_THT:C_Disc_D5.1mm_W3.2mm_P5.00mm, F.Cu at (262.2, 22.8)
- added C2: 0.1uF, Capacitor_THT:C_Disc_D5.1mm_W3.2mm_P5.00mm, F.Cu at (122.2, 136.7)
- added C2: 0.1uF, Capacitor_THT:C_Disc_D5.1mm_W3.2mm_P5.00mm, F.Cu at (262.2, 136.7)
- added C2: 0.1uF, Capacitor_THT:C_Disc_D5.1mm_W3.2mm_P5.00mm, F.Cu at (262.2, 31.7)
- added J1: Screw_Terminal_01x04 (buttons), TerminalBlock_Phoenix:TerminalBlock_Phoenix_MKDS-1,5-4-5.08_1x04_P5.08mm_Horizontal, F.Cu at (124.7, 167.2)
- added J1: Screw_Terminal_01x04 (buttons), TerminalBlock_Phoenix:TerminalBlock_Phoenix_MKDS-1,5-4-5.08_1x04_P5.08mm_Horizontal, F.Cu at (264.7, 167.2)
- added J1: Screw_Terminal_01x04 (buttons), TerminalBlock_Phoenix:TerminalBlock_Phoenix_MKDS-1,5-4-5.08_1x04_P5.08mm_Horizontal, F.Cu at (264.7, 62.1)
- added J2: Conn_01x06_Male (programmer), Connector_PinHeader_2.54mm:PinHeader_1x06_P2.54mm_Vertical, F.Cu at (82.8, 204.0)
- added J2: Conn_01x06_Male (programmer), Connector_PinHeader_2.54mm:PinHeader_1x06_P2.54mm_Vertical, F.Cu at (222.8, 204.0)
- added J2: Conn_01x06_Male (programmer), Connector_PinHeader_2.54mm:PinHeader_1x06_P2.54mm_Vertical, F.Cu at (222.8, 99.0)
- added J3: Screw_Terminal_01x06 (output), TerminalBlock_Phoenix:TerminalBlock_Phoenix_MKDS-1,5-6-5.08_1x06_P5.08mm_Horizontal, F.Cu at (35.8, 186.2)
- added J3: Screw_Terminal_01x06 (output), TerminalBlock_Phoenix:TerminalBlock_Phoenix_MKDS-1,5-6-5.08_1x06_P5.08mm_Horizontal, F.Cu at (175.8, 186.2)
- added J3: Screw_Terminal_01x06 (output), TerminalBlock_Phoenix:TerminalBlock_Phoenix_MKDS-1,5-6-5.08_1x06_P5.08mm_Horizontal, F.Cu at (175.8, 81.2)
- added J4: Conn_01x02_Male (i2c), Connector_PinHeader_2.54mm:PinHeader_1x02_P2.54mm_Vertical, F.Cu at (98.0, 143.7)
- added J4: Conn_01x02_Male (i2c), Connector_PinHeader_2.54mm:PinHeader_1x02_P2.54mm_Vertical, F.Cu at (238.0, 143.7)
- added J4: Conn_01x02_Male (i2c), Connector_PinHeader_2.54mm:PinHeader_1x02_P2.54mm_Vertical, F.Cu at (238.0, 38.7)
- added J5: Conn_01x02_Male (Jumper), Connector_PinHeader_2.54mm:PinHeader_1x02_P2.54mm_Vertical, F.Cu at (76.4, 204.0)
- added J5: Conn_01x02_Male (Jumper), Connector_PinHeader_2.54mm:PinHeader_1x02_P2.54mm_Vertical, F.Cu at (216.4, 204.0)
- added J5: Conn_01x02_Male (Jumper), Connector_PinHeader_2.54mm:PinHeader_1x02_P2.54mm_Vertical, F.Cu at (216.4, 99.0)
- added J6: Conn_01x03_Male (Indicators), Connector_PinHeader_2.54mm:PinHeader_1x03_P2.54mm_Vertical, F.Cu at (71.4, 146.8)
- added J6: Conn_01x03_Male (Indicators), Connector_PinHeader_2.54mm:PinHeader_1x03_P2.54mm_Vertical, F.Cu at (211.4, 146.8)
- added J6: Conn_01x03_Male (Indicators), Connector_PinHeader_2.54mm:PinHeader_1x03_P2.54mm_Vertical, F.Cu at (211.4, 41.8)
- added J7: Screw_Terminal_01x02 (power), TerminalBlock_Phoenix:TerminalBlock_Phoenix_MKDS-1,5-2_1x02_P5.00mm_Horizontal, F.Cu at (94.2, 129.1)
- added J7: Screw_Terminal_01x02 (power), TerminalBlock_Phoenix:TerminalBlock_Phoenix_MKDS-1,5-2_1x02_P5.00mm_Horizontal, F.Cu at (234.2, 129.1)
- added J7: Screw_Terminal_01x02 (power), TerminalBlock_Phoenix:TerminalBlock_Phoenix_MKDS-1,5-2_1x02_P5.00mm_Horizontal, F.Cu at (234.2, 24.1)
- added Q1: IRF8308M, scheme:IRF840, F.Cu at (48.5, 188.7)
- added Q1: IRF8308M, scheme:IRF840, F.Cu at (188.5, 188.7)
- added Q1: IRF8308M, scheme:IRF840, F.Cu at (188.5, 83.7)
- added Q2: IRF8308M, scheme:IRF840, F.Cu at (48.5, 174.8)
- added Q2: IRF8308M, scheme:IRF840, F.Cu at (188.5, 174.8)
- added Q2: IRF8308M, scheme:IRF840, F.Cu at (188.5, 69.8)
- added Q3: IRF8308M, scheme:IRF840, F.Cu at (48.5, 160.8)
- added Q3: IRF8308M, scheme:IRF840, F.Cu at (188.5, 160.8)
- added Q3: IRF8308M, scheme:IRF840, F.Cu at (188.5, 55.8)
- added R1: 10K, Resistor_THT:R_Axial_DIN0207_L6.3mm_D2.5mm_P7.62mm_Horizontal, F.Cu at (98.0, 188.1)
- added R1: 10K, Resistor_THT:R_Axial_DIN0207_L6.3mm_D2.5mm_P7.62mm_Horizontal, F.Cu at (238.0, 188.1)
- added R1: 10K, Resistor_THT:R_Axial_DIN0207_L6.3mm_D2.5mm_P7.62mm_Horizontal, F.Cu at (238.0, 83.1)
- added R10: 10K, Resistor_THT:R_Axial_DIN0207_L6.3mm_D2.5mm_P7.62mm_Horizontal, F.Cu at (56.1, 162.1)
- added R10: 10K, Resistor_THT:R_Axial_DIN0207_L6.3mm_D2.5mm_P7.62mm_Horizontal, F.Cu at (196.1, 162.1)
- added R10: 10K, Resistor_THT:R_Axial_DIN0207_L6.3mm_D2.5mm_P7.62mm_Horizontal, F.Cu at (196.1, 57.1)
- added R2: 220Ohm, Resistor_THT:R_Axial_DIN0207_L6.3mm_D2.5mm_P7.62mm_Horizontal, F.Cu at (103.1, 164.0)
- added R2: 220Ohm, Resistor_THT:R_Axial_DIN0207_L6.3mm_D2.5mm_P7.62mm_Horizontal, F.Cu at (243.1, 164.0)
- added R2: 220Ohm, Resistor_THT:R_Axial_DIN0207_L6.3mm_D2.5mm_P7.62mm_Horizontal, F.Cu at (243.1, 59.0)
- added R3: 220Ohm, Resistor_THT:R_Axial_DIN0207_L6.3mm_D2.5mm_P7.62mm_Horizontal, F.Cu at (103.1, 158.3)
- added R3: 220Ohm, Resistor_THT:R_Axial_DIN0207_L6.3mm_D2.5mm_P7.62mm_Horizontal, F.Cu at (243.1, 158.3)
- added R3: 220Ohm, Resistor_THT:R_Axial_DIN0207_L6.3mm_D2.5mm_P7.62mm_Horizontal, F.Cu at (243.1, 53.3)
- added R4: 220Ohm, Resistor_THT:R_Axial_DIN0207_L6.3mm_D2.5mm_P7.62mm_Horizontal, F.Cu at (103.1, 153.2)
- added R4: 220Ohm, Resistor_THT:R_Axial_DIN0207_L6.3mm_D2.5mm_P7.62mm_Horizontal, F.Cu at (243.1, 153.2)
- added R4: 220Ohm, Resistor_THT:R_Axial_DIN0207_L6.3mm_D2.5mm_P7.62mm_Horizontal, F.Cu at (243.1, 48.2)
- added R5: 10K, Resistor_THT:R_Axial_DIN0207_L6.3mm_D2.5mm_P7.62mm_Horizontal, F.Cu at (56.1, 190.0)
- added R5: 10K, Resistor_THT:R_Axial_DIN0207_L6.3mm_D2.5mm_P7.62mm_Horizontal, F.Cu at (196.1, 190.0)
- added R5: 10K, Resistor_THT:R_Axial_DIN0207_L6.3mm_D2.5mm_P7.62mm_Horizontal, F.Cu at (196.1, 85.0)
- added R6: 100Ohm, Resistor_THT:R_Axial_DIN0207_L6.3mm_D2.5mm_P7.62mm_Horizontal, F.Cu at (59.9, 197.6)
- added R6: 100Ohm, Resistor_THT:R_Axial_DIN0207_L6.3mm_D2.5mm_P7.62mm_Horizontal, F.Cu at (199.9, 197.6)
- added R6: 100Ohm, Resistor_THT:R_Axial_DIN0207_L6.3mm_D2.5mm_P7.62mm_Horizontal, F.Cu at (199.9, 92.6)
- added R7: 100Ohm, Resistor_THT:R_Axial_DIN0207_L6.3mm_D2.5mm_P7.62mm_Horizontal, F.Cu at (70.1, 173.5)
- added R7: 100Ohm, Resistor_THT:R_Axial_DIN0207_L6.3mm_D2.5mm_P7.62mm_Horizontal, F.Cu at (210.1, 173.5)
- added R7: 100Ohm, Resistor_THT:R_Axial_DIN0207_L6.3mm_D2.5mm_P7.62mm_Horizontal, F.Cu at (210.1, 68.5)
- added R8: 10K, Resistor_THT:R_Axial_DIN0207_L6.3mm_D2.5mm_P7.62mm_Horizontal, F.Cu at (56.1, 176.0)
- added R8: 10K, Resistor_THT:R_Axial_DIN0207_L6.3mm_D2.5mm_P7.62mm_Horizontal, F.Cu at (196.1, 176.0)
- added R8: 10K, Resistor_THT:R_Axial_DIN0207_L6.3mm_D2.5mm_P7.62mm_Horizontal, F.Cu at (196.1, 71.0)
- added R9: 100Ohm, Resistor_THT:R_Axial_DIN0207_L6.3mm_D2.5mm_P7.62mm_Horizontal, F.Cu at (70.1, 162.1)
- added R9: 100Ohm, Resistor_THT:R_Axial_DIN0207_L6.3mm_D2.5mm_P7.62mm_Horizontal, F.Cu at (210.1, 162.1)
- added R9: 100Ohm, Resistor_THT:R_Axial_DIN0207_L6.3mm_D2.5mm_P7.62mm_Horizontal, F.Cu at (210.1, 57.1)
- added SW1: SW_Push (reset), Button_Switch_THT:SW_PUSH_6mm, F.Cu at (71.4, 187.5)
- added SW1: SW_Push (reset), Button_Switch_THT:SW_PUSH_6mm, F.Cu at (211.4, 187.5)
- added SW1: SW_Push (reset), Button_Switch_THT:SW_PUSH_6mm, F.Cu at (211.4, 82.5)
- added U1: L7805, Package_TO_SOT_THT:TO-220-3_Vertical, F.Cu at (109.5, 129.1)
- added U1: L7805, Package_TO_SOT_THT:TO-220-3_Vertical, F.Cu at (249.5, 129.1)
- added U1: L7805, Package_TO_SOT_THT:TO-220-3_Vertical, F.Cu at (249.5, 24.1)
- added U2: ATmega8A-PU, Package_DIP:DIP-28_W7.62mm, F.Cu at (82.6, 148.4)
- added U2: ATmega8A-PU, Package_DIP:DIP-28_W7.62mm, F.Cu at (222.6, 148.4)
- added U2: ATmega8A-PU, Package_DIP:DIP-28_W7.62mm, F.Cu at (222.6, 43.4)
- moved J6 25.5 mm to (71.4, 41.8)
- moved SW1 25.5 mm to (71.4, 82.5)
- moved R10 25.5 mm to (56.1, 57.1)
- moved R5 25.5 mm to (56.1, 85.0)
- moved R8 25.5 mm to (56.1, 71.0)
- moved C1 25.5 mm to (122.2, 22.8)
- moved C2 25.5 mm to (122.2, 31.7)
- moved J1 25.5 mm to (124.7, 62.1)
- moved J2 25.5 mm to (82.8, 99.0)
- moved J3 25.5 mm to (35.8, 81.2)
- moved J5 25.5 mm to (76.4, 99.0)
- moved J7 25.5 mm to (94.2, 24.1)
- moved R1 25.5 mm to (98.0, 83.1)
- moved R2 25.5 mm to (103.1, 59.0)
- moved R3 25.5 mm to (103.1, 53.3)
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Routing:
- net (no net): track 3460.8 -> 3761.0 mm, vias 0 -> 12
- net Net-(C2-Pad2): track 239.1 -> 271.3 mm
- net GND: track 258.7 -> 289.1 mm, vias 0 -> 4
- net Net-(R9-Pad2): track 23.1 -> 33.1 mm
- net Net-(R7-Pad2): track 15.8 -> 23.3 mm
- net Net-(J4-Pad1): track 7.89 -> 14.0 mm
- net Net-(J4-Pad2): track 7.89 -> 13.7 mm
- net Net-(J2-Pad4): track 44.8 -> 48.4 mm
- net Net-(J2-Pad3): track 188.9 -> 191.1 mm
- net Net-(J2-Pad6): track 34.9 -> 36.4 mm
- net Net-(J6-Pad3): track 13.0 -> 13.7 mm
Other:
- net class Default: clearance 0.2 -> 0.4
- rule trace_clearance: 0.2 -> 0.4

Commit message: scheme: Get rid of second layer
Parts:
- removed the C1 at (122.2, 127.8)
- removed the C1 at (262.2, 127.8)
- removed the C1 at (262.2, 22.8)
- removed the C2 at (122.2, 136.7)
- removed the C2 at (262.2, 136.7)
- removed the C2 at (262.2, 31.7)
- removed the J1 at (124.7, 167.2)
- removed the J1 at (264.7, 167.2)
- removed the J1 at (264.7, 62.1)
- removed the J2 at (82.8, 204.0)
- removed the J2 at (222.8, 204.0)
- removed the J2 at (222.8, 99.0)
- removed the J3 at (35.8, 186.2)
- removed the J3 at (175.8, 186.2)
- removed the J3 at (175.8, 81.2)
- removed the J4 at (98.0, 143.7)
- removed the J4 at (238.0, 143.7)
- removed the J4 at (238.0, 38.7)
- removed the J5 at (76.4, 204.0)
- removed the J5 at (216.4, 204.0)
- removed the J5 at (216.4, 99.0)
- removed the J6 at (71.4, 146.8)
- removed the J6 at (211.4, 146.8)
- removed the J6 at (211.4, 41.8)
- removed the J7 at (94.2, 129.1)
- removed the J7 at (234.2, 129.1)
- removed the J7 at (234.2, 24.1)
- removed the Q1 at (48.5, 188.7)
- removed the Q1 at (188.5, 188.7)
- removed the Q1 at (188.5, 83.7)
- removed the Q2 at (48.5, 174.8)
- removed the Q2 at (188.5, 174.8)
- removed the Q2 at (188.5, 69.8)
- removed the Q3 at (48.5, 160.8)
- removed the Q3 at (188.5, 160.8)
- removed the Q3 at (188.5, 55.8)
- removed the R1 at (98.0, 188.1)
- removed the R1 at (238.0, 188.1)
- removed the R1 at (238.0, 83.1)
- removed the R10 at (56.1, 162.1)
- removed the R10 at (196.1, 162.1)
- removed the R10 at (196.1, 57.1)
- removed the R2 at (103.1, 164.0)
- removed the R2 at (243.1, 164.0)
- removed the R2 at (243.1, 59.0)
- removed the R3 at (103.1, 158.3)
- removed the R3 at (243.1, 158.3)
- removed the R3 at (243.1, 53.3)
- removed the R4 at (103.1, 153.2)
- removed the R4 at (243.1, 153.2)
- removed the R4 at (243.1, 48.2)
- removed the R5 at (56.1, 190.0)
- removed the R5 at (196.1, 190.0)
- removed the R5 at (196.1, 85.0)
- removed the R6 at (59.9, 197.6)
- removed the R6 at (199.9, 197.6)
- removed the R6 at (199.9, 92.6)
- removed the R7 at (70.1, 173.5)
- removed the R7 at (210.1, 173.5)
- removed the R7 at (210.1, 68.5)
- removed the R8 at (56.1, 176.0)
- removed the R8 at (196.1, 176.0)
- removed the R8 at (196.1, 71.0)
- removed the R9 at (70.1, 162.1)
- removed the R9 at (210.1, 162.1)
- removed the R9 at (210.1, 57.1)
- removed the SW1 at (71.4, 187.5)
- removed the SW1 at (211.4, 187.5)
- removed the SW1 at (211.4, 82.5)
- removed the U1 at (109.5, 129.1)
- removed the U1 at (249.5, 129.1)
- removed the U1 at (249.5, 24.1)
- removed the U2 at (82.6, 148.4)
- removed the U2 at (222.6, 148.4)
- removed the U2 at (222.6, 43.4)
- added C1: 3.3uF, Capacitor_THT:C_Disc_D5.1mm_W3.2mm_P5.00mm, F.Cu at (227.2, 122.8)
- added C1: 3.3uF, Capacitor_THT:C_Disc_D5.1mm_W3.2mm_P5.00mm, F.Cu at (227.2, 17.8)
- added C1: 3.3uF, Capacitor_THT:C_Disc_D5.1mm_W3.2mm_P5.00mm, F.Cu at (97.2, 122.8)
- added C2: 0.1uF, Capacitor_THT:C_Disc_D5.1mm_W3.2mm_P5.00mm, F.Cu at (227.2, 131.7)
- added C2: 0.1uF, Capacitor_THT:C_Disc_D5.1mm_W3.2mm_P5.00mm, F.Cu at (227.2, 26.7)
- added C2: 0.1uF, Capacitor_THT:C_Disc_D5.1mm_W3.2mm_P5.00mm, F.Cu at (97.2, 131.7)
- added J1: Screw_Terminal_01x04 (buttons), TerminalBlock_Phoenix:TerminalBlock_Phoenix_MKDS-1,5-4-5.08_1x04_P5.08mm_Horizontal, F.Cu at (229.7, 162.2)
- added J1: Screw_Terminal_01x04 (buttons), TerminalBlock_Phoenix:TerminalBlock_Phoenix_MKDS-1,5-4-5.08_1x04_P5.08mm_Horizontal, F.Cu at (229.7, 57.1)
- added J1: Screw_Terminal_01x04 (buttons), TerminalBlock_Phoenix:TerminalBlock_Phoenix_MKDS-1,5-4-5.08_1x04_P5.08mm_Horizontal, F.Cu at (99.7, 162.2)
- added J2: Conn_01x06_Male (programmer), Connector_PinHeader_2.54mm:PinHeader_1x06_P2.54mm_Vertical, F.Cu at (187.8, 199.0)
- added J2: Conn_01x06_Male (programmer), Connector_PinHeader_2.54mm:PinHeader_1x06_P2.54mm_Vertical, F.Cu at (187.8, 94.0)
- added J2: Conn_01x06_Male (programmer), Connector_PinHeader_2.54mm:PinHeader_1x06_P2.54mm_Vertical, F.Cu at (57.8, 199.0)
- added J3: Screw_Terminal_01x06 (output), TerminalBlock_Phoenix:TerminalBlock_Phoenix_MKDS-1,5-6-5.08_1x06_P5.08mm_Horizontal, F.Cu at (140.8, 181.2)
- added J3: Screw_Terminal_01x06 (output), TerminalBlock_Phoenix:TerminalBlock_Phoenix_MKDS-1,5-6-5.08_1x06_P5.08mm_Horizontal, F.Cu at (140.8, 76.2)
- added J3: Screw_Terminal_01x06 (output), TerminalBlock_Phoenix:TerminalBlock_Phoenix_MKDS-1,5-6-5.08_1x06_P5.08mm_Horizontal, F.Cu at (10.8, 181.2)
- added J4: Conn_01x02_Male (i2c), Connector_PinHeader_2.54mm:PinHeader_1x02_P2.54mm_Vertical, F.Cu at (203.0, 138.7)
- added J4: Conn_01x02_Male (i2c), Connector_PinHeader_2.54mm:PinHeader_1x02_P2.54mm_Vertical, F.Cu at (203.0, 33.7)
- added J4: Conn_01x02_Male (i2c), Connector_PinHeader_2.54mm:PinHeader_1x02_P2.54mm_Vertical, F.Cu at (73.0, 138.7)
- added J5: Conn_01x02_Male (Jumper), Connector_PinHeader_2.54mm:PinHeader_1x02_P2.54mm_Vertical, F.Cu at (181.4, 199.0)
- added J5: Conn_01x02_Male (Jumper), Connector_PinHeader_2.54mm:PinHeader_1x02_P2.54mm_Vertical, F.Cu at (181.4, 94.0)
- added J5: Conn_01x02_Male (Jumper), Connector_PinHeader_2.54mm:PinHeader_1x02_P2.54mm_Vertical, F.Cu at (51.4, 199.0)
- added J6: Conn_01x03_Male (Indicators), Connector_PinHeader_2.54mm:PinHeader_1x03_P2.54mm_Vertical, F.Cu at (176.4, 141.8)
- added J6: Conn_01x03_Male (Indicators), Connector_PinHeader_2.54mm:PinHeader_1x03_P2.54mm_Vertical, F.Cu at (176.4, 36.8)
- added J6: Conn_01x03_Male (Indicators), Connector_PinHeader_2.54mm:PinHeader_1x03_P2.54mm_Vertical, F.Cu at (46.4, 141.8)
- added J7: Screw_Terminal_01x02 (power), TerminalBlock_Phoenix:TerminalBlock_Phoenix_MKDS-1,5-2_1x02_P5.00mm_Horizontal, F.Cu at (199.2, 124.0)
- added J7: Screw_Terminal_01x02 (power), TerminalBlock_Phoenix:TerminalBlock_Phoenix_MKDS-1,5-2_1x02_P5.00mm_Horizontal, F.Cu at (199.2, 19.1)
- added J7: Screw_Terminal_01x02 (power), TerminalBlock_Phoenix:TerminalBlock_Phoenix_MKDS-1,5-2_1x02_P5.00mm_Horizontal, F.Cu at (69.2, 124.0)
- added Q1: IRF8308M, scheme:IRF840, F.Cu at (153.5, 183.7)
- added Q1: IRF8308M, scheme:IRF840, F.Cu at (153.5, 78.7)
- added Q1: IRF8308M, scheme:IRF840, F.Cu at (23.5, 183.7)
- added Q2: IRF8308M, scheme:IRF840, F.Cu at (153.5, 169.8)
- added Q2: IRF8308M, scheme:IRF840, F.Cu at (153.5, 64.8)
- added Q2: IRF8308M, scheme:IRF840, F.Cu at (23.5, 169.8)
- added Q3: IRF8308M, scheme:IRF840, F.Cu at (153.5, 155.8)
- added Q3: IRF8308M, scheme:IRF840, F.Cu at (153.5, 50.8)
- added Q3: IRF8308M, scheme:IRF840, F.Cu at (23.5, 155.8)
- added R1: 10K, Resistor_THT:R_Axial_DIN0207_L6.3mm_D2.5mm_P7.62mm_Horizontal, F.Cu at (203.0, 183.1)
- added R1: 10K, Resistor_THT:R_Axial_DIN0207_L6.3mm_D2.5mm_P7.62mm_Horizontal, F.Cu at (203.0, 78.1)
- added R1: 10K, Resistor_THT:R_Axial_DIN0207_L6.3mm_D2.5mm_P7.62mm_Horizontal, F.Cu at (73.0, 183.1)
- added R10: 10K, Resistor_THT:R_Axial_DIN0207_L6.3mm_D2.5mm_P7.62mm_Horizontal, F.Cu at (161.1, 157.1)
- added R10: 10K, Resistor_THT:R_Axial_DIN0207_L6.3mm_D2.5mm_P7.62mm_Horizontal, F.Cu at (161.1, 52.1)
- added R10: 10K, Resistor_THT:R_Axial_DIN0207_L6.3mm_D2.5mm_P7.62mm_Horizontal, F.Cu at (31.1, 157.1)
- added R2: 220Ohm, Resistor_THT:R_Axial_DIN0207_L6.3mm_D2.5mm_P7.62mm_Horizontal, F.Cu at (208.0, 147.3)
- added R2: 220Ohm, Resistor_THT:R_Axial_DIN0207_L6.3mm_D2.5mm_P7.62mm_Horizontal, F.Cu at (208.0, 42.3)
- added R2: 220Ohm, Resistor_THT:R_Axial_DIN0207_L6.3mm_D2.5mm_P7.62mm_Horizontal, F.Cu at (78.0, 147.3)
- added R3: 220Ohm, Resistor_THT:R_Axial_DIN0207_L6.3mm_D2.5mm_P7.62mm_Horizontal, F.Cu at (213.9, 147.2)
- added R3: 220Ohm, Resistor_THT:R_Axial_DIN0207_L6.3mm_D2.5mm_P7.62mm_Horizontal, F.Cu at (213.9, 42.2)
- added R3: 220Ohm, Resistor_THT:R_Axial_DIN0207_L6.3mm_D2.5mm_P7.62mm_Horizontal, F.Cu at (83.9, 147.2)
- added R4: 220Ohm, Resistor_THT:R_Axial_DIN0207_L6.3mm_D2.5mm_P7.62mm_Horizontal, F.Cu at (220.3, 147.2)
- added R4: 220Ohm, Resistor_THT:R_Axial_DIN0207_L6.3mm_D2.5mm_P7.62mm_Horizontal, F.Cu at (220.3, 42.2)
- added R4: 220Ohm, Resistor_THT:R_Axial_DIN0207_L6.3mm_D2.5mm_P7.62mm_Horizontal, F.Cu at (90.3, 147.2)
- added R5: 10K, Resistor_THT:R_Axial_DIN0207_L6.3mm_D2.5mm_P7.62mm_Horizontal, F.Cu at (161.1, 185.0)
- added R5: 10K, Resistor_THT:R_Axial_DIN0207_L6.3mm_D2.5mm_P7.62mm_Horizontal, F.Cu at (161.1, 80.0)
- added R5: 10K, Resistor_THT:R_Axial_DIN0207_L6.3mm_D2.5mm_P7.62mm_Horizontal, F.Cu at (31.1, 185.0)
- added R6: 100Ohm, Resistor_THT:R_Axial_DIN0207_L6.3mm_D2.5mm_P7.62mm_Horizontal, F.Cu at (164.9, 192.6)
- added R6: 100Ohm, Resistor_THT:R_Axial_DIN0207_L6.3mm_D2.5mm_P7.62mm_Horizontal, F.Cu at (164.9, 87.6)
- added R6: 100Ohm, Resistor_THT:R_Axial_DIN0207_L6.3mm_D2.5mm_P7.62mm_Horizontal, F.Cu at (34.9, 192.6)
- added R7: 100Ohm, Resistor_THT:R_Axial_DIN0207_L6.3mm_D2.5mm_P7.62mm_Horizontal, F.Cu at (175.1, 168.5)
- added R7: 100Ohm, Resistor_THT:R_Axial_DIN0207_L6.3mm_D2.5mm_P7.62mm_Horizontal, F.Cu at (175.1, 63.5)
- added R7: 100Ohm, Resistor_THT:R_Axial_DIN0207_L6.3mm_D2.5mm_P7.62mm_Horizontal, F.Cu at (45.1, 168.5)
- added R8: 10K, Resistor_THT:R_Axial_DIN0207_L6.3mm_D2.5mm_P7.62mm_Horizontal, F.Cu at (161.1, 171.0)
- added R8: 10K, Resistor_THT:R_Axial_DIN0207_L6.3mm_D2.5mm_P7.62mm_Horizontal, F.Cu at (161.1, 66.0)
- added R8: 10K, Resistor_THT:R_Axial_DIN0207_L6.3mm_D2.5mm_P7.62mm_Horizontal, F.Cu at (31.1, 171.0)
- added R9: 100Ohm, Resistor_THT:R_Axial_DIN0207_L6.3mm_D2.5mm_P7.62mm_Horizontal, F.Cu at (175.1, 157.1)
- added R9: 100Ohm, Resistor_THT:R_Axial_DIN0207_L6.3mm_D2.5mm_P7.62mm_Horizontal, F.Cu at (175.1, 52.1)
- added R9: 100Ohm, Resistor_THT:R_Axial_DIN0207_L6.3mm_D2.5mm_P7.62mm_Horizontal, F.Cu at (45.1, 157.1)
- added SW1: SW_Push (reset), Button_Switch_THT:SW_PUSH_6mm, F.Cu at (176.4, 182.5)
- added SW1: SW_Push (reset), Button_Switch_THT:SW_PUSH_6mm, F.Cu at (176.4, 77.5)
- added SW1: SW_Push (reset), Button_Switch_THT:SW_PUSH_6mm, F.Cu at (46.4, 182.5)
- added U1: L7805, Package_TO_SOT_THT:TO-220-3_Vertical, F.Cu at (214.5, 124.0)
- added U1: L7805, Package_TO_SOT_THT:TO-220-3_Vertical, F.Cu at (214.5, 19.1)
- added U1: L7805, Package_TO_SOT_THT:TO-220-3_Vertical, F.Cu at (84.5, 124.0)
- added U2: ATmega8A-PU, Package_DIP:DIP-28_W7.62mm, F.Cu at (187.6, 143.4)
- added U2: ATmega8A-PU, Package_DIP:DIP-28_W7.62mm, F.Cu at (187.6, 38.4)
- added U2: ATmega8A-PU, Package_DIP:DIP-28_W7.62mm, F.Cu at (57.6, 143.4)
- moved R2 30.2 mm to (78.0, 42.3), turned to 270 degrees
- moved J6 25.5 mm to (46.4, 36.8)
- moved SW1 25.5 mm to (46.4, 77.5)
- moved R10 25.5 mm to (31.1, 52.1)
- moved R5 25.5 mm to (31.1, 80.0)
- moved R8 25.5 mm to (31.1, 66.0)
- moved C1 25.5 mm to (97.2, 17.8)
- moved C2 25.5 mm to (97.2, 26.7)
- moved J1 25.5 mm to (99.7, 57.1)
- moved J2 25.5 mm to (57.8, 94.0)
- moved J3 25.5 mm to (10.8, 76.2)
- moved J4 25.5 mm to (73.0, 33.7)
- moved J5 25.5 mm to (51.4, 94.0)
- moved J7 25.5 mm to (69.2, 19.1)
- moved R1 25.5 mm to (73.0, 78.1)
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Routing:
- net (no net): track 3761.0 -> 3671.5 mm, vias 12 -> 0
- net GND: track 289.1 -> 259.4 mm, vias 4 -> 0
- net Net-(J1-Pad1): track 41.4 -> 44.3 mm
- net Net-(J1-Pad2): track 41.0 -> 38.5 mm
